Commit message: refactor(description): ♻️ Match bero.urdf to robot's real size
- adjust model size based on measurements
- correct LiDAR and IMU sensor positions and orientations
- add a supporting frame and box for the LiDAR

File: src/bero_description/urdf/bero.urdf (robot description, URDF)
Before this commit: robot bero, 9 links, 8 joints
Links:
- added link imu_link; visual box size=0.005 0.01 0.002
- added link laser_base_link; visual box size=0.05 0.05 0.025
- added link laser_frame_bl; visual cylinder length=0.028 radius=0.0025
- added link laser_frame_br; visual cylinder length=0.028 radius=0.0025
- added link laser_frame_fl; visual cylinder length=0.028 radius=0.0025
- added link laser_frame_fr; visual cylinder length=0.028 radius=0.0025
- link base_link: geometry visual cylinder length=0.044 radius=0.145
- link laser: mass 0.1 -> None; geometry visual cylinder length=0.018 radius=0.025
- link lower_frame: geometry visual cylinder length=0.05 radius=0.01; visual cylinder length=0.05 radius=0.01
- link plate_link: geometry visual cylinder length=0.014 radius=0.12
- link upper_frame: geometry visual cylinder length=0.164 radius=0.01; visual cylinder length=0.164 radius=0.01
- link upper_link: geometry visual cylinder length=0.001 radius=0.115
- link wheel_link_back: mass 1.0 -> None; geometry visual cylinder length=0.021 radius=0.041
- link wheel_link_left: mass 1.0 -> None; geometry visual cylinder length=0.021 radius=0.041
- link wheel_link_right: mass 1.0 -> None; geometry visual cylinder length=0.021 radius=0.041
Joints:
- added joint imu_joint: type fixed, parent upper_link, child imu_link, origin xyz=0.0 0.0 0.0015 rpy=0 0 -1.5708
- added joint laser_base_joint: type fixed, parent upper_link, child laser_base_link, origin xyz=0.03 0.0 0.041
- added joint pillar_joint_bl: type fixed, parent upper_link, child laser_frame_bl, origin xyz=0.005 0.025 0.0145
- added joint pillar_joint_br: type fixed, parent upper_link, child laser_frame_br, origin xyz=0.005 -0.025 0.0145
- added joint pillar_joint_fl: type fixed, parent upper_link, child laser_frame_fl, origin xyz=0.055 0.025 0.0145
- added joint pillar_joint_fr: type fixed, parent upper_link, child laser_frame_fr, origin xyz=0.055 -0.025 0.0145
- joint laser_joint: origin xyz=0.05 0.0 0.12 rpy=0.0 0.0 3.14159 -> xyz=0.0 0.0 0.0215 rpy=0.0 0.0 3.14159; parent upper_link -> laser_base_link
- joint lower_joint: origin xyz=0.0 0.0 0.1 rpy=0.0 0.0 0.0 -> xyz=0.0 0.0 0.047 rpy=0.0 0.0 0.0
- joint plate_joint: origin xyz=0.0 0.0 -0.05 rpy=0.0 0.0 0.0 -> xyz=0.0 0.0 0.032 rpy=0.0 0.0 0.0
- joint top_joint: origin xyz=0.0 0.0 -0.05 rpy=0.0 0.0 0.0 -> xyz=0.0 0.0 0.0825 rpy=0.0 0.0 0.0
- joint upper_joint: origin xyz=0.0 0.0 0.15 rpy=0.0 0.0 0.0 -> xyz=0.0 0.0 0.089 rpy=0.0 0.0 0.0
- joint wheel_joint_back: origin xyz=-0.1465 0.0 0.05 rpy=0.0 1.5708 3.14159 -> xyz=-0.1465 0.0 -0.007 rpy=0.0 1.5708 3.14159
- joint wheel_joint_left: origin xyz=0.07325 0.1269 0.05 rpy=1.5708 0 -0.5236 -> xyz=0.07325 0.1269 -0.007 rpy=1.5708 0 -0.5236
- joint wheel_joint_right: origin xyz=0.07325 -0.1269 0.05 rpy=1.5708 0 0.5236 -> xyz=0.07325 -0.1269 -0.007 rpy=1.5708 0 0.5236

Commit message: fix(description): 🐛 Add base_footprint to prevent sinking issue in map (#28)
- bero.urdf: add base_footprint link and raise base_link by 0.048 m (fixed joint)
- ekf_odom.yaml: set ekf base frame to base_footprint
- mapper_params_online_async.yaml: set mapping base frame to base_footprint

File: src/bero_description/urdf/bero.urdf (robot description, URDF)
Before this commit: robot bero, 15 links, 14 joints
Links:
- added link base_footprint
Joints:
- added joint base_footprint_joint: type fixed, parent base_footprint, child base_link, origin xyz=0 0 0.048 rpy=0 0 0
